Commit message: add IMU sensor on the model and set correct installion position

File: prius_description/urdf/prius.urdf (robot description, URDF)
Before this commit: robot prius, 24 links, 23 joints
Links:
- added link imu_link, mass 1
Joints:
- added joint imu_joint: type fixed, parent chassis, child imu_link, origin xyz=0 0 0 rpy=0 0 -1.5707
